File: hardware/thefly.brd (EAGLE design)
At the start: 54 x 54 mm, 31 parts, among them IC1 AP7313-1.8, J1 54-00298, U1 SGTL5000XNLA3, U2 MAX4466EXK

Commit message: elec layout progress
Parts:
- added C12: 100n, thefly:0603-CAP
- moved C11 115.7 mm to (30.9, 44.6), turned to 180 degrees
- moved R8 108.1 mm to (30.9, 42.6)
- moved C10 107.8 mm to (29.9, 39.7), turned to 270 degrees
- moved R7 102.8 mm to (31.9, 39.7), turned to 90 degrees
- moved R6 101.6 mm to (38.2, 38.9)
- moved R5 100.7 mm to (38.2, 40.9), turned to 180 degrees
- moved C9 99.8 mm to (38.2, 42.9), turned to 180 degrees
- moved C8 98.5 mm to (32.4, 46.9), turned to 180 degrees
- moved R4 94.8 mm to (35.0, 44.9), turned to 180 degrees
- moved R3 93.5 mm to (38.2, 44.9), turned to 180 degrees
- moved R9 83.0 mm to (29.6, 7.30), turned to 270 degrees
- moved L2 78.9 mm to (35.0, 36.2), turned to 90 degrees
- moved L3 78.1 mm to (32.0, 33.8), turned to 90 degrees
- moved R2 58.0 mm to (43.6, 4.60), turned to 180 degrees
- moved C5 55.9 mm to (37.4, 20.7)
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Connections:
- net AGND: now also C12.2
- net BCLK: now also JP1.15; no longer JP1.21
- net HP-L: now also U1.1; no longer U1.4
- net HP-R: now also U1.4; no longer U1.1
- net MCLK: now also JP1.16; no longer JP1.19
- net N$2: now also C12.1
Routing:
- net 3.3V: track 0.00 -> 90.0 mm, vias 0 -> 6
- net HP-SENSE-L: track 0.00 -> 82.4 mm, vias 0 -> 1
- net HP-MIC: track 0.00 -> 51.7 mm, vias 0 -> 2
- net SDA: track 0.00 -> 35.8 mm, vias 0 -> 2
- net I2S_DIN: track 0.00 -> 34.2 mm, vias 0 -> 2
- net N$4: track 0.00 -> 31.4 mm
- net LRCLK: track 0.00 -> 29.2 mm
- net SCL: track 0.00 -> 26.8 mm, vias 0 -> 2
- net MIC2: track 0.00 -> 23.6 mm, vias 0 -> 2
- net BCLK: track 0.00 -> 23.5 mm
- net N$5: track 0.00 -> 20.5 mm
- net I2S_DOUT: track 0.00 -> 20.4 mm, vias 0 -> 2
- net HP-GND: track 0.00 -> 18.8 mm
- net HP-R: track 0.00 -> 17.7 mm
- net N$2: track 0.00 -> 15.7 mm, vias 0 -> 2
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- added copper zone on layer 1, net AGND
- added copper zone on layer 16, net AGND
- added copper zone on layer 1, net GND
- added copper zone on layer 16, net GND

Commit message: elec layout wip
Routing:
- net GND: vias 87 -> 90

Commit message: more pcb work
Parts:
- added C13: 100n, thefly:0603-CAP
- added MIC2: 3SM122KZB1VD-002-R, thefly:MIC_3SM122KZB1VD-002-R
- moved R9 0.25 mm to (29.6, 7.55)
Connections:
- removed net N$10: C9.1, MIC1.P, R3.1
- removed net N$2: C12.1, L2.2, R4.2, R6.2, U2.5
- new net MICRAW: C9.1, MIC1.P, MIC2.2, R3.1
- new net VCCA2: C12.1, C13.2, L2.2, MIC2.1, R4.2, R6.2, U2.5
- net AGND: now also C13.1, MIC2.3_1, MIC2.3_2
Routing:
- net VCCA2: track 0.00 -> 24.9 mm, vias 0 -> 3
- net MICRAW: track 0.00 -> 17.3 mm, vias 0 -> 2
- net N$2: track 15.5 -> 0.00 mm, vias 2 -> 0
- net N$10: track 7.56 -> 0.00 mm
- net AGND: track 0.00 -> 1.01 mm, vias 27 -> 36
- net GND: vias 90 -> 107

Commit message: pcb layout wip
Parts:
- added C14: 100n, thefly:0603-CAP
- added L4: 600, thefly:0603
- added U$5: THE-FLY-LOGO, thefly:THE-FLY-LOGO
- moved R2 2.02 mm to (43.3, 6.60)
Connections:
- new net N$1: C14.1, L4.2, R2.1
- net 3.3V: now also L4.1; no longer R2.1
- net GND: now also C14.2
Routing:
- net N$1: track 0.00 -> 4.80 mm
- net HP-MIC: track 51.7 -> 49.7 mm
- net N$4: track 31.4 -> 29.9 mm
- net 3.3V: track 90.2 -> 91.6 mm
- net HP-SENSE-L: track 82.3 -> 81.2 mm
- net GND: vias 107 -> 113
- net AGND: vias 36 -> 35
Other:
- board text added: "20260605A"

Commit message: pcb wip
Parts:
- moved R9 0.20 mm to (29.6, 7.35)
Routing:
- net HP-SENSE-L: track 81.2 -> 87.2 mm
- net 3.3V: track 91.6 -> 89.1 mm
- net GND: vias 113 -> 103

Commit message: pcb wip
Parts:
- J1: value 54-00298 -> 54-00298-HOLES; device thefly:TENSILITY_54-00298 -> thefly:TENSILITY_54-00298_HOLES
Routing:
- net 3.3V: track 89.1 -> 88.5 mm
- net GND: vias 103 -> 110
Changed lines of the file:
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@@
 <attribute name="VALUE" x="37.303790625" y="20.897590625" size="0.8128" layer="27" font="vector" rot="R90"/>
 </element>
-<element name="J1" library="thefly" package="TENSILITY_54-00298" value="54-00298" x="34" y="7" smashed="yes">
-<attribute name="DESCRIPTION" value="                                                      Connector, 4C audio jack, 3.5xL14 mm, thru hole, gold plated                                              " x="34" y="7" size="1.778" layer="27" display="off"/>
-<attribute name="SNAPEDA_LINK" value="https://www.snapeda.com/parts/54-00298/Tensility/view-part/?ref=snap" x="34" y="7" size="1.778" layer="27" display="off"/>
-<attribute name="MF" value="Tensility International Corp" x="34" y="7" size="1.778" layer="27" display="off"/>
-<attribute name="PACKAGE" value="None" x="34" y="7" size="1.778" layer="27" display="off"/>
-<attribute name="MP" value="54-00298" x="34" y="7" size="1.778" layer="27" display="off"/>
-<attribute name="DIGIKEY_PART_NUMBER" value="839-54-00298CT-ND" x="34" y="7" size="1.778" layer="27" display="off"/>
-<attribute name="CHECK_PRICES" value="https://www.snapeda.com/parts/54-00298/Tensility/view-part/?ref=eda" x="34" y="7" size="1.778" layer="27" display="off"/>
+<element name="J1" library="thefly" package="TENSILITY_54-00298_HOLES" value="54-00298-HOLES" x="34" y="7" smashed="yes">
 <attribute name="VALUE" x="30.6" y="15" size="0.8128" layer="27" font="vector"/>
 </element>
@@
 </element>
 <element name="R2" library="thefly" package="0603-RES" value="1M" x="43.3" y="6.6" smashed="yes" rot="R180">
-<attribute name="NAME" x="42.911" y="7.462" size="0.8128" layer="25" font="vector"/>
+<attribute name="NAME" x="45.011" y="6.262" size="0.8128" layer="25" font="vector"/>
 <attribute name="VALUE" x="44.316" y="7.743" size="0.8128" layer="27" font="vector" rot="R180"/>
 </element>
@@
 <via x="51.2" y="41" extent="1-16" drill="0.3" shape="octagon"/>
 <via x="51.2" y="38.4" extent="1-16" drill="0.3" shape="octagon"/>
-<via x="34.4" y="8.6" extent="1-16" drill="0.3" shape="octagon"/>
 <contactref element="C14" pad="2"/>
 <via x="45.6" y="2.1" extent="1-16" drill="0.3" shape="octagon"/>
@@
 <via x="42.1" y="15.6" extent="1-16" drill="0.3" shape="octagon"/>
 <via x="27.5" y="14.7" extent="1-16" drill="0.3" shape="octagon"/>
+<via x="37.8" y="2.5" extent="1-16" drill="0.3" shape="octagon"/>
+<via x="30.9" y="2.2" extent="1-16" drill="0.3" shape="octagon"/>
+<via x="30" y="1.2" extent="1-16" drill="0.3" shape="octagon"/>
+<via x="31.1" y="6.5" extent="1-16" drill="0.3" shape="octagon"/>
+<via x="37.8" y="6.4" extent="1-16" drill="0.3" shape="octagon"/>
+<via x="34.4" y="8.6" extent="1-16" drill="0.3" shape="octagon"/>
+<via x="35.2" y="7.2" extent="1-16" drill="0.3" shape="octagon"/>
+<via x="33.2" y="5.2" extent="1-16" drill="0.3" shape="octagon"/>
 </signal>
 <signal name="HP-L">
@@
 <wire x1="32.3" y1="15.2" x2="31.5" y2="15.2" width="0.2032" layer="1"/>
 <wire x1="31.5" y1="15.2" x2="30.9" y2="14.6" width="0.2032" layer="1"/>
-<wire x1="30.9" y1="14.6" x2="30.9" y2="11.85" width="0.2032" layer="1"/>
-<wire x1="30.9" y1="11.85" x2="31.45" y2="11.3" width="0.2032" layer="1"/>
+<wire x1="30.9" y1="14.6" x2="30.9" y2="12.35" width="0.2032" layer="1"/>
+<wire x1="30.9" y1="12.35" x2="31.45" y2="11.3" width="0.2032" layer="1"/>
 </signal>
 <signal name="HP-GND">
@@
 <wire x1="33.3" y1="20.3" x2="33.3" y2="14.9" width="0.2032" layer="1"/>
 <wire x1="33.3" y1="14.9" x2="35.1" y2="13.1" width="0.2032" layer="1"/>
-<wire x1="35.1" y1="13.1" x2="35.1" y2="10.3" width="0.2032" layer="1"/>
-<wire x1="35.1" y1="10.3" x2="31.8" y2="7" width="0.2032" layer="1"/>
-<wire x1="31.8" y1="7" x2="31.8" y2="4.9" width="0.2032" layer="1"/>
+<wire x1="35.1" y1="13.1" x2="35.1" y2="8.2" width="0.2032" layer="1"/>
+<wire x1="35.1" y1="8.2" x2="31.8" y2="4.9" width="0.2032" layer="1"/>
 </signal>
 <signal name="HP-SENSE-L">
 <contactref element="J1" pad="5"/>
 <contactref element="R9" pad="1"/>
-<wire x1="32.7" y1="13" x2="32.7" y2="10.1" width="0.2032" layer="1"/>
-<wire x1="32.7" y1="10.1" x2="31.4" y2="8.8" width="0.2032" layer="1"/>
-<wire x1="31.4" y1="8.8" x2="30.2" y2="8.8" width="0.2032" layer="1"/>
-<wire x1="32.2" y1="13.5" x2="32.7" y2="13" width="0.2032" layer="16"/>
-<wire x1="32.7" y1="13" x2="32.7" y2="7.9" width="0.2032" layer="16"/>
+<wire x1="32.7" y1="12.5" x2="32.7" y2="10.1" width="0.2032" layer="1"/>
+<wire x1="32.7" y1="10.1" x2="31.2" y2="8.6" width="0.2032" layer="1"/>
+<wire x1="31.2" y1="8.6" x2="30" y2="8.6" width="0.2032" layer="1"/>
+<wire x1="32.2" y1="13.5" x2="32.7" y2="12.5" width="0.2032" layer="16"/>
+<wire x1="32.7" y1="12.5" x2="32.7" y2="7.9" width="0.2032" layer="16"/>
 <wire x1="46.4" y1="10.8" x2="50.5" y2="14.9" width="0.2032" layer="16"/>
 <wire x1="50.5" y1="14.9" x2="50.5" y2="42.497809375" width="0.2032" layer="16"/>
@@
 <wire x1="32" y1="7.2" x2="30.8" y2="7.2" width="0.2032" layer="16"/>
 <wire x1="30.8" y1="7.2" x2="30" y2="6.4" width="0.2032" layer="16"/>
-<wire x1="30.2" y1="8.8" x2="29.6" y2="8.2" width="0.2032" layer="1"/>
-<wire x1="32.7" y1="13" x2="32.2" y2="13.5" width="0.2032" layer="1"/>
+<wire x1="30" y1="8.6" x2="29.6" y2="8.2" width="0.2032" layer="1"/>
+<wire x1="32.7" y1="12.5" x2="32.2" y2="13.5" width="0.2032" layer="1"/>
 </signal>
 <signal name="HP-SENSE-R">
@@
 <wire x1="45.3" y1="4.6" x2="44.15" y2="4.6" width="0.2032" layer="1"/>
 <wire x1="45.3" y1="4.6" x2="43.7" y2="3" width="0.254" layer="16"/>
-<wire x1="43.7" y1="3" x2="38.3" y2="3" width="0.254" layer="16"/>
-<wire x1="38.3" y1="3" x2="38.3" y2="9.3" width="0.254" layer="16"/>
+<wire x1="43.7" y1="3" x2="39.3" y2="3" width="0.254" layer="16"/>
+<wire x1="39.3" y1="3" x2="38.5" y2="3.8" width="0.254" layer="16"/>
+<wire x1="38.5" y1="3.8" x2="38.5" y2="9.1" width="0.254" layer="16"/>
 <via x="28.7" y="15.2" extent="1-16" drill="0.3" shape="octagon"/>
-<wire x1="38.3" y1="9.3" x2="38" y2="9.6" width="0.254" layer="16"/>
-<wire x1="38" y1="9.6" x2="38" y2="14" width="0.254" layer="16"/>
-<wire x1="38" y1="14" x2="36.8" y2="15.2" width="0.254" layer="16"/>
+<wire x1="38.5" y1="9.1" x2="38.2" y2="9.4" width="0.254" layer="16"/>
+<wire x1="38.2" y1="9.4" x2="38.2" y2="13.8" width="0.254" layer="16"/>
+<wire x1="38.2" y1="13.8" x2="36.8" y2="15.2" width="0.254" layer="16"/>
 <wire x1="29.6" y1="6.5" x2="28.7" y2="7.4" width="0.2032" layer="1"/>
 <wire x1="28.7" y1="7.4" x2="28.7" y2="15.2" width="0.2032" layer="1"/>

Commit message: progress on ext codec
Connections:
- net MCLK: now also JP1.13; no longer JP1.16
Routing:
- net MCLK: track 13.7 -> 19.9 mm, vias 0 -> 2
Other:
- board text added: "20260606A"
- board text removed: "20260605A"
Changed lines of the file:
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@@
 <board>
 <plain>
-<text x="9" y="48" size="1.27" layer="21" font="vector" ratio="10" align="top-left">20260605A</text>
+<text x="9" y="48" size="1.27" layer="21" font="vector" ratio="10" align="top-left">20260606A</text>
 </plain>
 <attributes>
@@
 <wire x1="34" y1="28.1" x2="34.4" y2="28.5" width="0.1524" layer="1"/>
 <wire x1="34.4" y1="28.5" x2="37.5" y2="28.5" width="0.1524" layer="1"/>
-<contactref element="JP1" pad="16"/>
 <wire x1="37.5" y1="28.5" x2="39" y2="27" width="0.1524" layer="1"/>
-<wire x1="39" y1="27" x2="43.36" y2="27" width="0.1524" layer="1"/>
+<contactref element="JP1" pad="13"/>
+<via x="39" y="27" extent="1-16" drill="0.3" shape="octagon"/>
+<wire x1="39" y1="27" x2="44.7" y2="27" width="0.2032" layer="16"/>
+<wire x1="44.7" y1="27" x2="47.24" y2="29.54" width="0.2032" layer="16"/>
+<via x="47.24" y="29.54" extent="1-16" drill="0.3" shape="octagon"/>
+<wire x1="47.24" y1="29.54" x2="48.44" y2="29.54" width="0.2032" layer="1"/>
 </signal>
 <signal name="VCCA2">

Commit message: more mclk pin shenanigans
Connections:
- net MCLK: now also JP1.14; no longer JP1.13
Routing:
- net MCLK: track 19.9 -> 16.6 mm
Changed lines of the file:
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@@
 <via x="33.91" y="19.32" extent="1-16" drill="0.3" shape="octagon"/>
 <via x="38.5" y="28.4" extent="1-16" drill="0.3" shape="octagon"/>
-<via x="41.2" y="27.6" extent="1-16" drill="0.3" shape="octagon"/>
+<via x="41.2" y="27.65" extent="1-16" drill="0.3" shape="octagon"/>
 <via x="50.6" y="44.8" extent="1-16" drill="0.3" shape="octagon"/>
 <via x="48.4" y="46" extent="1-16" drill="0.3" shape="octagon"/>
@@
 <wire x1="34.4" y1="28.5" x2="37.5" y2="28.5" width="0.1524" layer="1"/>
 <wire x1="37.5" y1="28.5" x2="39" y2="27" width="0.1524" layer="1"/>
-<contactref element="JP1" pad="13"/>
 <via x="39" y="27" extent="1-16" drill="0.3" shape="octagon"/>
-<wire x1="39" y1="27" x2="44.7" y2="27" width="0.2032" layer="16"/>
-<wire x1="44.7" y1="27" x2="47.24" y2="29.54" width="0.2032" layer="16"/>
-<via x="47.24" y="29.54" extent="1-16" drill="0.3" shape="octagon"/>
-<wire x1="47.24" y1="29.54" x2="48.44" y2="29.54" width="0.2032" layer="1"/>
+<wire x1="39" y1="27" x2="41.7" y2="27" width="0.2032" layer="16"/>
+<wire x1="41.7" y1="27" x2="44.24" y2="29.54" width="0.2032" layer="16"/>
+<via x="44.24" y="29.54" extent="1-16" drill="0.3" shape="octagon"/>
+<contactref element="JP1" pad="14"/>
+<wire x1="44.24" y1="29.54" x2="43.36" y2="29.54" width="0.2032" layer="1"/>
 </signal>
 <signal name="VCCA2">
