File: hardware/thefly.sch (EAGLE design)
At the start: 31 parts, among them IC1 AP7313-1.8, J1 54-00298, U1 SGTL5000XNLA3, U2 MAX4466EXK

Commit message: elec layout progress
Parts:
- added C12: 100n, thefly:CAP0603-CAP
Connections:
- net AGND: now also C12.2
- net BCLK: now also JP1.15; no longer JP1.21
- net HP-L: now also U1.HP_R; no longer U1.HP_L
- net HP-R: now also U1.HP_L; no longer U1.HP_R
- net MCLK: now also JP1.16; no longer JP1.19
- net N$2: now also C12.1

Commit message: elec layout wip
Changed lines of the file:
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@@
 <pinref part="JP1" gate="A" pin="2"/>
 <wire x1="160.02" y1="-40.64" x2="144.78" y2="-40.64" width="0.1524" layer="91"/>
+<junction x="160.02" y="-40.64"/>
 </segment>
 </net>

Commit message: more pcb work
Parts:
- added C13: 100n, thefly:CAP0603-CAP
- added MIC2: 3SM122KZB1VD-002-R, thefly:3SM122KZB1VD-002-R
Connections:
- removed net N$10: C9.1, MIC1.+, R3.1
- removed net N$2: C12.1, L2.P$2, R4.2, R6.2, U2.VCC
- new net MICRAW: C9.1, MIC1.+, MIC2.OUTPUT, R3.1
- new net VCCA2: C12.1, C13.2, L2.P$2, MIC2.VDD, R4.2, R6.2, U2.VCC
- net AGND: now also C13.1, MIC2.GND
Other:
- moved on the sheet: MIC1
Changed lines of the file:
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@@
 <part name="C12" library="thefly" deviceset="CAP" device="0603-CAP" value="100n"/>
 <part name="AGND6" library="thefly" deviceset="AGND" device=""/>
+<part name="MIC2" library="thefly" deviceset="3SM122KZB1VD-002-R" device=""/>
+<part name="AGND7" library="thefly" deviceset="AGND" device=""/>
+<part name="C13" library="thefly" deviceset="CAP" device="0603-CAP" value="100n"/>
+<part name="AGND8" library="thefly" deviceset="AGND" device=""/>
 </parts>
 <sheets>
@@
 <instance part="J1" gate="G$1" x="68.58" y="-38.1"/>
 <instance part="U2" gate="A" x="210.82" y="73.66"/>
-<instance part="MIC1" gate="G$1" x="154.94" y="71.12"/>
+<instance part="MIC1" gate="G$1" x="154.94" y="66.04" smashed="yes">
+<attribute name="NAME" x="156.21" y="62.23" size="1.778" layer="95"/>
+<attribute name="VALUE" x="156.21" y="60.325" size="1.778" layer="96"/>
+</instance>
 <instance part="U$2" gate="G$1" x="0" y="7.62"/>
 <instance part="IC1" gate="G$1" x="68.58" y="91.44"/>
@@
 <instance part="C8" gate="G$1" x="139.7" y="86.36"/>
 <instance part="AGND1" gate="VR1" x="233.68" y="55.88"/>
-<instance part="AGND2" gate="VR1" x="152.4" y="55.88"/>
+<instance part="AGND2" gate="VR1" x="152.4" y="53.34"/>
 <instance part="C9" gate="G$1" x="170.18" y="78.74" rot="R90"/>
 <instance part="R5" gate="G$1" x="180.34" y="71.12" rot="R90"/>
@@
 <instance part="C11" gate="G$1" x="190.5" y="27.94" rot="R180"/>
 <instance part="AGND4" gate="VR1" x="190.5" y="17.78"/>
-<instance part="AGND5" gate="VR1" x="139.7" y="73.66"/>
+<instance part="AGND5" gate="VR1" x="139.7" y="78.74"/>
 <instance part="GND1" gate="1" x="121.92" y="-35.56"/>
 <instance part="P+5" gate="G$1" x="172.72" y="-50.8"/>
@@
 <instance part="C12" gate="G$1" x="241.3" y="93.98" rot="R90"/>
 <instance part="AGND6" gate="VR1" x="246.38" y="88.9"/>
+<instance part="MIC2" gate="G$1" x="220.98" y="12.7"/>
+<instance part="AGND7" gate="VR1" x="236.22" y="-2.54"/>
+<instance part="C13" gate="G$1" x="236.22" y="25.4"/>
+<instance part="AGND8" gate="VR1" x="228.6" y="27.94"/>
 </instances>
 <busses>
@@
 </segment>
 </net>
-<net name="N$2" class="0">
+<net name="VCCA2" class="0">
 <segment>
 <pinref part="U2" gate="A" pin="VCC"/>
@@
 <wire x1="233.68" y1="81.28" x2="233.68" y2="93.98" width="0.1524" layer="91"/>
 <pinref part="R6" gate="G$1" pin="2"/>
-<wire x1="233.68" y1="93.98" x2="180.34" y2="93.98" width="0.1524" layer="91"/>
+<wire x1="233.68" y1="93.98" x2="231.14" y2="93.98" width="0.1524" layer="91"/>
+<wire x1="231.14" y1="93.98" x2="180.34" y2="93.98" width="0.1524" layer="91"/>
 <wire x1="180.34" y1="93.98" x2="180.34" y2="91.44" width="0.1524" layer="91"/>
 <pinref part="R4" gate="G$1" pin="2"/>
@@
 <wire x1="236.22" y1="93.98" x2="233.68" y2="93.98" width="0.1524" layer="91"/>
 <junction x="233.68" y="93.98"/>
+<wire x1="231.14" y1="93.98" x2="231.14" y2="99.06" width="0.1524" layer="91"/>
+<wire x1="231.14" y1="99.06" x2="228.6" y2="99.06" width="0.1524" layer="91"/>
+<junction x="231.14" y="93.98"/>
+<label x="228.6" y="99.06" size="1.27" layer="95" rot="R180" xref="yes"/>
+</segment>
+<segment>
+<pinref part="MIC2" gate="G$1" pin="VDD"/>
+<wire x1="233.68" y1="17.78" x2="236.22" y2="17.78" width="0.1524" layer="91"/>
+<wire x1="236.22" y1="17.78" x2="236.22" y2="20.32" width="0.1524" layer="91"/>
+<wire x1="236.22" y1="20.32" x2="238.76" y2="20.32" width="0.1524" layer="91"/>
+<label x="238.76" y="20.32" size="1.27" layer="95" xref="yes"/>
+<pinref part="C13" gate="G$1" pin="2"/>
+<wire x1="236.22" y1="22.86" x2="236.22" y2="20.32" width="0.1524" layer="91"/>
+<junction x="236.22" y="20.32"/>
 </segment>
 </net>
@@
 <pinref part="AGND5" gate="VR1" pin="AGND"/>
 <pinref part="C8" gate="G$1" pin="2"/>
-<wire x1="139.7" y1="76.2" x2="139.7" y2="83.82" width="0.1524" layer="91"/>
+<wire x1="139.7" y1="81.28" x2="139.7" y2="83.82" width="0.1524" layer="91"/>
 </segment>
 <segment>
 <pinref part="AGND2" gate="VR1" pin="AGND"/>
 <pinref part="MIC1" gate="G$1" pin="-"/>
-<wire x1="152.4" y1="58.42" x2="152.4" y2="66.04" width="0.1524" layer="91"/>
+<wire x1="152.4" y1="55.88" x2="152.4" y2="60.96" width="0.1524" layer="91"/>
 </segment>
 <segment>
@@
 <wire x1="243.84" y1="93.98" x2="246.38" y2="93.98" width="0.1524" layer="91"/>
 <wire x1="246.38" y1="93.98" x2="246.38" y2="91.44" width="0.1524" layer="91"/>
+</segment>
+<segment>
+<pinref part="MIC2" gate="G$1" pin="GND"/>
+<pinref part="AGND7" gate="VR1" pin="AGND"/>
+<wire x1="233.68" y1="7.62" x2="236.22" y2="7.62" width="0.1524" layer="91"/>
+<wire x1="236.22" y1="7.62" x2="236.22" y2="0" width="0.1524" layer="91"/>
+</segment>
+<segment>
+<pinref part="AGND8" gate="VR1" pin="AGND"/>
+<wire x1="228.6" y1="30.48" x2="228.6" y2="33.02" width="0.1524" layer="91"/>
+<pinref part="C13" gate="G$1" pin="1"/>
+<wire x1="228.6" y1="33.02" x2="236.22" y2="33.02" width="0.1524" layer="91"/>
+<wire x1="236.22" y1="33.02" x2="236.22" y2="30.48" width="0.1524" layer="91"/>
 </segment>
 </net>
@@
 </segment>
 </net>
-<net name="N$10" class="0">
-<segment>
-<pinref part="MIC1" gate="G$1" pin="+"/>
-<pinref part="R3" gate="G$1" pin="1"/>
-<wire x1="152.4" y1="76.2" x2="152.4" y2="78.74" width="0.1524" layer="91"/>
-<pinref part="C9" gate="G$1" pin="1"/>
-<wire x1="152.4" y1="78.74" x2="152.4" y2="81.28" width="0.1524" layer="91"/>
-<wire x1="152.4" y1="78.74" x2="165.1" y2="78.74" width="0.1524" layer="91"/>
-<junction x="152.4" y="78.74"/>
-</segment>
-</net>
 <net name="N$11" class="0">
 <segment>
@@
 </segment>
 </net>
+<net name="MICRAW" class="0">
+<segment>
+<label x="251.46" y="12.7" size="1.27" layer="95" xref="yes"/>
+<pinref part="MIC2" gate="G$1" pin="OUTPUT"/>
+<wire x1="251.46" y1="12.7" x2="233.68" y2="12.7" width="0.1524" layer="91"/>
+</segment>
+<segment>
+<pinref part="MIC1" gate="G$1" pin="+"/>
+<pinref part="R3" gate="G$1" pin="1"/>
+<wire x1="152.4" y1="71.12" x2="152.4" y2="76.2" width="0.1524" layer="91"/>
+<pinref part="C9" gate="G$1" pin="1"/>
+<wire x1="152.4" y1="76.2" x2="152.4" y2="78.74" width="0.1524" layer="91"/>
+<wire x1="152.4" y1="78.74" x2="152.4" y2="81.28" width="0.1524" layer="91"/>
+<wire x1="152.4" y1="78.74" x2="165.1" y2="78.74" width="0.1524" layer="91"/>
+<junction x="152.4" y="78.74"/>
+<wire x1="152.4" y1="76.2" x2="149.86" y2="76.2" width="0.1524" layer="91"/>
+<label x="149.86" y="76.2" size="1.27" layer="95" rot="R180" xref="yes"/>
+<junction x="152.4" y="76.2"/>
+</segment>
+</net>

Commit message: pcb layout wip
Parts:
- added C14: 100n, thefly:CAP0603-CAP
- added L4: 600, thefly:FB
- added U$5: THE-FLY-LOGO, thefly:THE-FLY-LOGO
Connections:
- new net N$1: C14.1, L4.P$2, R2.1
- net 3.3V: now also L4.P$1; no longer R2.1
- net GND: now also C14.2
Other:
- moved on the sheet: R2
Changed lines of the file:
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@@
 <part name="C13" library="thefly" deviceset="CAP" device="0603-CAP" value="100n"/>
 <part name="AGND8" library="thefly" deviceset="AGND" device=""/>
+<part name="L4" library="thefly" deviceset="FB" device="" value="600"/>
+<part name="C14" library="thefly" deviceset="CAP" device="0603-CAP" value="100n"/>
+<part name="GND11" library="thefly" deviceset="GND" device=""/>
+<part name="U$5" library="thefly" deviceset="THE-FLY-LOGO" device=""/>
 </parts>
 <sheets>
@@
 <instance part="R1" gate="G$1" x="129.54" y="5.08"/>
 <instance part="C7" gate="G$1" x="129.54" y="12.7" rot="R90"/>
-<instance part="R2" gate="G$1" x="121.92" y="-5.08" rot="R90"/>
-<instance part="P+3" gate="G$1" x="129.54" y="-10.16"/>
+<instance part="R2" gate="G$1" x="129.54" y="-2.54" rot="R180"/>
+<instance part="P+3" gate="G$1" x="170.18" y="0"/>
 <instance part="L2" gate="G$1" x="256.54" y="81.28"/>
 <instance part="L3" gate="G$1" x="241.3" y="66.04"/>
@@
 <instance part="C13" gate="G$1" x="236.22" y="25.4"/>
 <instance part="AGND8" gate="VR1" x="228.6" y="27.94"/>
+<instance part="L4" gate="G$1" x="162.56" y="-2.54"/>
+<instance part="C14" gate="G$1" x="149.86" y="-10.16"/>
+<instance part="GND11" gate="1" x="149.86" y="-17.78"/>
+<instance part="U$5" gate="G$1" x="-2.54" y="20.32"/>
 </instances>
 <busses>
@@
 <junction x="129.54" y="-43.18"/>
 </segment>
+<segment>
+<pinref part="C14" gate="G$1" pin="2"/>
+<pinref part="GND11" gate="1" pin="GND"/>
+<wire x1="149.86" y1="-12.7" x2="149.86" y2="-15.24" width="0.1524" layer="91"/>
+</segment>
 </net>
 <net name="1.8V" class="0">
@@
 </segment>
 <segment>
-<pinref part="P+3" gate="G$1" pin="3.3V"/>
-<wire x1="129.54" y1="-10.16" x2="129.54" y2="-12.7" width="0.1524" layer="91"/>
-<wire x1="129.54" y1="-12.7" x2="121.92" y2="-12.7" width="0.1524" layer="91"/>
-<pinref part="R2" gate="G$1" pin="1"/>
-<wire x1="121.92" y1="-12.7" x2="121.92" y2="-10.16" width="0.1524" layer="91"/>
-</segment>
-<segment>
 <pinref part="L2" gate="G$1" pin="P$1"/>
 <pinref part="P+4" gate="G$1" pin="3.3V"/>
@@
 <pinref part="R9" gate="G$1" pin="2"/>
 <wire x1="160.02" y1="-25.4" x2="160.02" y2="-27.94" width="0.1524" layer="91"/>
+</segment>
+<segment>
+<pinref part="P+3" gate="G$1" pin="3.3V"/>
+<wire x1="170.18" y1="0" x2="170.18" y2="-2.54" width="0.1524" layer="91"/>
+<pinref part="L4" gate="G$1" pin="P$1"/>
+<wire x1="170.18" y1="-2.54" x2="167.64" y2="-2.54" width="0.1524" layer="91"/>
 </segment>
 </net>
@@
 <wire x1="109.22" y1="2.54" x2="109.22" y2="5.08" width="0.1524" layer="91"/>
 <pinref part="R2" gate="G$1" pin="2"/>
-<wire x1="121.92" y1="0" x2="121.92" y2="5.08" width="0.1524" layer="91"/>
+<wire x1="124.46" y1="-2.54" x2="121.92" y2="-2.54" width="0.1524" layer="91"/>
+<wire x1="121.92" y1="-2.54" x2="121.92" y2="5.08" width="0.1524" layer="91"/>
 <junction x="121.92" y="5.08"/>
 <junction x="109.22" y="5.08"/>
@@
 </segment>
 </net>
+<net name="N$1" class="0">
+<segment>
+<pinref part="R2" gate="G$1" pin="1"/>
+<pinref part="L4" gate="G$1" pin="P$2"/>
+<wire x1="157.48" y1="-2.54" x2="149.86" y2="-2.54" width="0.1524" layer="91"/>
+<pinref part="C14" gate="G$1" pin="1"/>
+<wire x1="149.86" y1="-2.54" x2="134.62" y2="-2.54" width="0.1524" layer="91"/>
+<wire x1="149.86" y1="-5.08" x2="149.86" y2="-2.54" width="0.1524" layer="91"/>
+<junction x="149.86" y="-2.54"/>
+</segment>
+</net>

Commit message: pcb wip
Parts:
- J1: value 54-00298 -> 54-00298-HOLES; device thefly:54-00298 -> thefly:54-00298-HOLES
Changed lines of the file:
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@@
 <part name="JP1" library="thefly" deviceset="PINHD-2X15" device="-SMD-R"/>
 <part name="U1" library="thefly" deviceset="SGTL5000XNLA3" device=""/>
-<part name="J1" library="thefly" deviceset="54-00298" device=""/>
+<part name="J1" library="thefly" deviceset="54-00298" device="-HOLES" value="54-00298-HOLES"/>
 <part name="U2" library="thefly" deviceset="MAX4466EXK" device=""/>
 <part name="MIC1" library="thefly" deviceset="POM-3535P-3-R" device=""/>

Commit message: progress on ext codec
Connections:
- net MCLK: now also JP1.13; no longer JP1.16
Changed lines of the file:
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@@
 </segment>
 <segment>
-<pinref part="JP1" gate="A" pin="16"/>
-<wire x1="144.78" y1="-58.42" x2="152.4" y2="-58.42" width="0.1524" layer="91"/>
-<label x="152.4" y="-58.42" size="1.27" layer="95" xref="yes"/>
+<pinref part="JP1" gate="A" pin="13"/>
+<wire x1="137.16" y1="-55.88" x2="129.54" y2="-55.88" width="0.1524" layer="91"/>
+<label x="129.54" y="-55.88" size="1.27" layer="95" rot="R180" xref="yes"/>
 </segment>
 </net>

Commit message: more mclk pin shenanigans
Connections:
- net MCLK: now also JP1.14; no longer JP1.13
Changed lines of the file:
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@@
 </segment>
 <segment>
-<pinref part="JP1" gate="A" pin="13"/>
-<wire x1="137.16" y1="-55.88" x2="129.54" y2="-55.88" width="0.1524" layer="91"/>
-<label x="129.54" y="-55.88" size="1.27" layer="95" rot="R180" xref="yes"/>
+<pinref part="JP1" gate="A" pin="14"/>
+<wire x1="144.78" y1="-55.88" x2="152.4" y2="-55.88" width="0.1524" layer="91"/>
+<label x="152.4" y="-55.88" size="1.27" layer="95" xref="yes"/>
 </segment>
 </net>
